File: LCD_board_STM32/LCD_board_STM32.kicad_pcb (KiCad board)
At the start: 2 copper layers, 48 x 43.5 mm, 74 parts, among them CON1 PIN-2x4, CON2 PIN-2x4, CON3 PIN-2x4, CON4 SWD-6pin, CON5 PIN-1x2, CON6 micro_sd, Q1 PDTC114ET, Q2 CSTCE, SW1 MicroswitchSmt6x4_V, SW2 MicroswitchSmt6x4_V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

Commit message: Working on circuit.
Parts:
- removed C10: C, 0805_M
- added C19: 100n, 0603_N, F.Cu at (79.4, 52.5)
- added C20: 100n, 0603_N, F.Cu at (87.5, 55.6)
- added C21: 100n, 0603_N, F.Cu at (91.8, 46.9)
- added C22: 100n, 0603_N, F.Cu at (83.0, 43.2)
- added C23: C, 0805_N, F.Cu at (81.9, 63.8)
- added C24: C, 0805_N, F.Cu at (85.1, 65.9)
- added C25: C, 0805_N, F.Cu at (51.6, 34.1)
- added C26: C, 0603_N, F.Cu at (91.1, 43.0)
- added Q3: FDC6331L, SOT23-6_N, F.Cu at (60.4, 34.1)
- added Q4: FDC6331L, SOT23-6_N, F.Cu at (60.4, 37.9)
- added Q5: FDC6331L, SOT23-6_N, F.Cu at (60.4, 41.7)
- added Q6: FDC6331L, SOT23-6_N, F.Cu at (60.4, 45.5)
- added R38: R, 0603_R_N, F.Cu at (79.4, 49.5)
- added R39: R, 0603_R_N, F.Cu at (91.1, 44.6)
- added R40: R, 0603_R_N, F.Cu at (91.8, 49.9)
- added R41: R, 0603_R_N, F.Cu at (88.1, 43.0)
- C18: footprint 0805_M -> 0805_N; moved to F.Cu
- C9: value C -> 100n; footprint 0805_M -> 0603_N; moved to F.Cu
- U3, U4: moved to F.Cu
- moved U1 41.8 mm to (85.6, 49.4)
- moved Q2 40.8 mm to (84.1, 56.1)
- moved C18 18.5 mm to (47.8, 34.1)
- moved C9 18.0 mm to (57.2, 61.9), turned to 90 degrees
- moved U4 17.0 mm to (59.9, 63.3), turned to 270 degrees
- moved U3 17.0 mm to (59.9, 60.5), turned to 270 degrees
- moved U5 2.18 mm to (49.7, 39.6), turned to 180 degrees
- moved U6 2.18 mm to (49.7, 39.6), turned to 270 degrees
- moved C6 0.08 mm to (61.0, 60.4)
- moved R12 0.08 mm to (52.1, 60.4)
- moved R9 0.08 mm to (56.5, 60.4)
- moved C8 0.07 mm to (61.0, 66.1)
- moved R16 0.07 mm to (52.1, 66.1)
- moved R24 0.06 mm to (47.6, 66.1)
- moved R14 0.06 mm to (56.5, 66.1)
Connections:
- U1 pad 17: (no net) -> Net-(R40-Pad2)
- U1 pad 25: (no net) -> Net-(C26-Pad1)
- U1 pad 35: (no net) -> GND
- U1 pad 36: (no net) -> VCC
- U1 pad 44: (no net) -> Net-(R38-Pad2)
Routing:
- net GND: track 7.73 -> 47.1 mm, vias 2 -> 6
- net VCC: track 5.08 -> 15.3 mm, vias 0 -> 6
- net PIN7: track 0.00 -> 10.1 mm
- net PIN11: track 0.00 -> 10.1 mm
- net PIN9: track 0.00 -> 10.1 mm
- net PIN2: track 3.12 -> 13.1 mm
- net PIN10: track 0.00 -> 10.0 mm
- net PIN8: track 0.00 -> 10.0 mm
- net PIN3: track 3.12 -> 13.1 mm
- net PIN6: track 0.00 -> 9.97 mm
- net PIN4: track 0.00 -> 9.94 mm
- net PIN5: track 0.00 -> 9.93 mm
- net uC10: track 0.00 -> 6.56 mm, vias 0 -> 1
- net uC6: track 0.00 -> 6.52 mm, vias 0 -> 1
- net uC2: track 0.00 -> 6.51 mm, vias 0 -> 1
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Other:
- net class Default: clearance 0.2 -> 0.153; trace_width 0.25 -> 0.153; via_dia 0.6 -> 0.51; via_drill 0.4 -> 0.3
- rule trace_clearance: 0.2 -> 0.153
- rule trace_min: 0.2 -> 0.153
- rule via_min_size: 0.4 -> 0.153

Commit message: Working on circuit.
Parts:
- moved C24 44.2 mm to (41.0, 62.4)
- moved C23 41.4 mm to (43.6, 48.0)
- moved C20 39.9 mm to (48.1, 62.2)
- moved C21 39.9 mm to (52.4, 53.5)
- moved R40 39.9 mm to (52.4, 56.5)
- moved C19 39.9 mm to (40.0, 59.1)
- moved R38 39.9 mm to (40.0, 56.1)
- moved C22 39.9 mm to (43.6, 49.8)
- moved C26 39.9 mm to (51.7, 49.6)
- moved Q2 39.9 mm to (44.7, 62.7)
- moved R39 39.9 mm to (51.7, 51.2)
- moved R41 39.9 mm to (48.7, 49.6)
- moved U1 39.9 mm to (46.2, 56.0)
- moved C9 1.70 mm to (58.0, 63.4)
- moved U3 1.00 mm to (60.9, 60.5)
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Connections:
- CON4 pad 6: SWO -> SWO/SCK
- D1 pad 2: (no net) -> Net-(D1-Pad2)
- R40 pad 1: (no net) -> uC7
- R41 pad 2: (no net) -> Net-(D1-Pad2)
- SW1 pad 2: (no net) -> SW1
- SW2 pad 2: (no net) -> SW2
- SW3 pad 2: (no net) -> SW3
- U1 pad 10: uC0 -> SW1
- U1 pad 18: uC7 -> uC8
- U1 pad 19: (no net) -> uC9
- U1 pad 2: (no net) -> TFT_CS
- U1 pad 20: (no net) -> SW3
- U1 pad 21: (no net) -> uC11
- U1 pad 38: (no net) -> SW2
- U1 pad 39: SWO -> SWO/SCK
- U1 pad 41: (no net) -> MOSI
- U1 pad 45: (no net) -> uC10
- U1 pad 46: (no net) -> uC0
- U2 pad 12: (no net) -> TFT_CS
- U2 pad 8: (no net) -> MOSI
- U2 pad 9: (no net) -> SWO/SCK
- U3 pad 4: PIN4 -> PIN5
- U3 pad 5: PIN5 -> PIN4
- U4 pad 4: PIN6 -> PIN7
- U4 pad 5: PIN7 -> PIN6
Routing:
- net GND: track 47.1 -> 66.4 mm
- net VPP: track 0.00 -> 15.0 mm
- net VCC: track 15.3 -> 28.7 mm
- net uC6: track 6.52 -> 19.3 mm
- net uC4: track 6.42 -> 15.6 mm
- net uC11: track 6.41 -> 13.1 mm
- net uC10: track 6.56 -> 13.0 mm
- net PIN11: track 10.1 -> 16.2 mm
- net uC9: track 6.29 -> 12.0 mm
- net uC8: track 6.45 -> 11.7 mm
- net PIN10: track 10.0 -> 15.0 mm
- net PIN9: track 10.1 -> 14.6 mm
- net PIN4: track 9.94 -> 14.0 mm
- net PIN7: track 10.1 -> 14.1 mm
- net PIN8: track 10.0 -> 14.0 mm
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- added copper zone on B.Cu, net GND

Commit message: Rename nets
Connections:
- C1 pad 1: PIN0 -> PIN4
- C11 pad 1: PIN8 -> PIN0
- C12 pad 1: PIN9 -> PIN1
- C13 pad 1: PIN10 -> PIN2
- C14 pad 1: PIN11 -> PIN3
- C2 pad 1: PIN1 -> PIN5
- C3 pad 1: PIN2 -> PIN6
- C4 pad 1: PIN3 -> PIN7
- C5 pad 1: PIN4 -> PIN8
- C6 pad 1: PIN5 -> PIN9
- C7 pad 1: PIN6 -> PIN10
- C8 pad 1: PIN7 -> PIN11
- CON1 pad 2: PIN8 -> PIN0
- CON1 pad 4: PIN9 -> PIN1
- CON1 pad 6: PIN10 -> PIN2
- CON1 pad 8: PIN11 -> PIN3
- CON2 pad 2: PIN0 -> PIN4
- CON2 pad 4: PIN1 -> PIN5
- CON2 pad 6: PIN2 -> PIN6
- CON2 pad 8: PIN3 -> PIN7
- CON3 pad 2: PIN4 -> PIN8
- CON3 pad 4: PIN5 -> PIN9
- CON3 pad 6: PIN6 -> PIN10
- CON3 pad 8: PIN7 -> PIN11
- Q3 pad 2: PIN8 -> PIN0
- Q3 pad 3: PIN8 -> PIN0
- Q3 pad 5: uC8 -> uC0
- Q4 pad 2: PIN9 -> PIN1
- Q4 pad 3: PIN9 -> PIN1
- Q4 pad 5: uC9 -> uC1
- Q5 pad 2: PIN10 -> PIN2
- Q5 pad 3: PIN10 -> PIN2
- Q5 pad 5: uC10 -> uC2
- Q6 pad 2: PIN11 -> PIN3
- Q6 pad 3: PIN11 -> PIN3
- Q6 pad 5: uC11 -> uC3
- R1 pad 1: PIN0 -> PIN4
- R10 pad 1: uC3 -> uC7
- R10 pad 2: PIN3 -> PIN7
- R11 pad 1: uC4 -> uC8
- R11 pad 2: PIN4 -> PIN8
- R12 pad 1: uC5 -> uC9
- R12 pad 2: PIN5 -> PIN9
- R13 pad 1: PIN6 -> PIN10
- R14 pad 1: PIN7 -> PIN11
- R15 pad 1: uC6 -> uC10
- R15 pad 2: PIN6 -> PIN10
- R16 pad 1: uC7 -> uC11
- R16 pad 2: PIN7 -> PIN11
- R17 pad 2: uC0 -> uC4
- R18 pad 2: uC1 -> uC5
- R19 pad 2: uC2 -> uC6
- R2 pad 1: PIN1 -> PIN5
- R20 pad 2: uC3 -> uC7
- R21 pad 2: uC4 -> uC8
- R22 pad 2: uC5 -> uC9
- R23 pad 2: uC6 -> uC10
- R24 pad 2: uC7 -> uC11
- R25 pad 1: PIN8 -> PIN0
- R26 pad 1: PIN9 -> PIN1
- R27 pad 1: PIN10 -> PIN2
- R28 pad 1: PIN11 -> PIN3
- R29 pad 1: uC8 -> uC0
- R29 pad 2: PIN8 -> PIN0
- R3 pad 1: PIN2 -> PIN6
- R30 pad 1: uC9 -> uC1
- R30 pad 2: PIN9 -> PIN1
- R31 pad 1: uC10 -> uC2
- R31 pad 2: PIN10 -> PIN2
- R32 pad 1: uC11 -> uC3
- R32 pad 2: PIN11 -> PIN3
- R33 pad 2: uC8 -> uC0
- R34 pad 2: uC9 -> uC1
- R35 pad 2: uC10 -> uC2
- R36 pad 2: uC11 -> uC3
- R4 pad 1: uC1 -> uC5
- R4 pad 2: PIN1 -> PIN5
- R40 pad 1: uC7 -> uC11
- R5 pad 1: uC0 -> uC4
- R5 pad 2: PIN0 -> PIN4
- R6 pad 1: uC2 -> uC6
- R6 pad 2: PIN2 -> PIN6
- R7 pad 1: PIN3 -> PIN7
- R8 pad 1: PIN4 -> PIN8
- R9 pad 1: PIN5 -> PIN9
- U1 pad 11: uC1 -> uC5
- U1 pad 12: uC2 -> uC6
- U1 pad 13: uC3 -> uC7
- U1 pad 14: uC4 -> uC8
- U1 pad 15: uC5 -> uC9
- U1 pad 16: uC6 -> uC10
- U1 pad 18: uC8 -> uC0
- U1 pad 19: uC9 -> uC1
- U1 pad 21: uC11 -> uC3
- U1 pad 45: uC10 -> uC2
- U1 pad 46: uC0 -> uC4
- U3 pad 4: PIN5 -> PIN9
- U3 pad 5: PIN4 -> PIN8
- U3 pad 6: uC4 -> uC8
- U4 pad 4: PIN7 -> PIN11
- U4 pad 5: PIN6 -> PIN10
- U4 pad 6: uC6 -> uC10
Routing:
- net uC6: track 19.3 -> 6.51 mm
- net uC4: track 15.6 -> 6.61 mm
- net uC3: track 6.37 -> 13.1 mm
- net uC11: track 13.1 -> 6.39 mm
- net uC2: track 6.51 -> 13.0 mm
- net uC10: track 13.0 -> 19.3 mm
- net uC9: track 12.0 -> 6.42 mm
- net uC1: track 6.54 -> 12.0 mm
- net uC0: track 6.61 -> 11.7 mm
- net uC8: track 11.7 -> 15.6 mm
- net PIN3: track 13.1 -> 16.2 mm
- net PIN10: track 15.0 -> 12.9 mm
- net PIN11: track 16.2 -> 14.1 mm
- net PIN2: track 13.1 -> 15.0 mm
- net PIN9: track 14.6 -> 12.9 mm
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